Commit message: Imported upstream version '2.0.0' of 'upstream'

File: open_manipulator_description/urdf/open_manipulator.gazebo.xacro (robot description, xacro)
@@ -1,81 +1,41 @@
 <?xml version="1.0"?>
-<robot>
+<robot xmlns:xacro="http://ros.org/wiki/xacro">
+  <!-- Gazebo Reference macro -->
+  <xacro:macro name="RefLink" params="ref">
+    <gazebo reference="${ref}">
+      <kp>1000000.0</kp>
+      <kd>100.0</kd>
+      <mu1>30.0</mu1>
+      <mu2>30.0</mu2>
+      <maxVel>1.0</maxVel>
+      <minDepth>0.001</minDepth>
+      <material>Gazebo/DarkGrey</material>
+    </gazebo>
+  </xacro:macro>
   <!-- World -->
   <gazebo reference="world">
   </gazebo>
   <!-- Link1 -->
-  <gazebo reference="link1">
-    <kp>1000000.0</kp>
-    <kd>100.0</kd>
-    <mu1>30.0</mu1>
-    <mu2>30.0</mu2>
-    <maxVel>1.0</maxVel>
-    <minDepth>0.001</minDepth>
-    <material>Gazebo/DarkGrey</material>
-  </gazebo>
+  <RefLink ref="link1"/>
   <!-- Link2 -->
-  <gazebo reference="link2">
-    <kp>1000000.0</kp>
-    <kd>100.0</kd>
-    <mu1>30.0</mu1>
-    <mu2>30.0</mu2>
-    <maxVel>1.0</maxVel>
-    <minDepth>0.001</minDepth>
-    <material>Gazebo/DarkGrey</material>
-  </gazebo>
+  <RefLink ref="link2"/>
   <!-- Link3 -->
-  <gazebo reference="link3">
-    <kp>1000000.0</kp>
-    <kd>100.0</kd>
-    <mu1>30.0</mu1>
-    <mu2>30.0</mu2>
-    <maxVel>1.0</maxVel>
-    <minDepth>0.001</minDepth>
-    <material>Gazebo/DarkGrey</material>
-  </gazebo>
+  <RefLink ref="link3"/>
   <!-- Link4 -->
-  <gazebo reference="link4">
-    <kp>1000000.0</kp>
-    <kd>100.0</kd>
-    <mu1>30.0</mu1>
-    <mu2>30.0</mu2>
-    <maxVel>1.0</maxVel>
-    <minDepth>0.001</minDepth>
-    <material>Gazebo/DarkGrey</material>
-  </gazebo>
+  <RefLink ref="link4"/>
   <!-- Link5 -->
-  <gazebo reference="link5">
-    <kp>1000000.0</kp>
-    <kd>100.0</kd>
-    <mu1>30.0</mu1>
-    <mu2>30.0</mu2>
-    <maxVel>1.0</maxVel>
-    <minDepth>0.001</minDepth>
-    <material>Gazebo/DarkGrey</material>
-  </gazebo>
-  <!-- grip_link -->
-  <gazebo reference="grip_link">
-    <kp>1000000.0</kp>
-    <kd>100.0</kd>
-    <mu1>30.0</mu1>
-    <mu2>30.0</mu2>
-    <maxVel>1.0</maxVel>
-    <minDepth>0.001</minDepth>
-    <material>Gazebo/DarkGrey</material>
-  </gazebo>
-  <!-- grip_link_sub -->
-  <gazebo reference="grip_link_sub">
-    <kp>1000000.0</kp>
-    <kd>100.0</kd>
-    <mu1>30.0</mu1>
-    <mu2>30.0</mu2>
-    <maxVel>1.0</maxVel>
-    <minDepth>0.001</minDepth>
-    <material>Gazebo/DarkGrey</material>
+  <RefLink ref="link5"/>
+  <!-- gripper_link -->
+  <RefLink ref="gripper_link"/>
+  <!-- gripper_link_sub -->
+  <RefLink ref="gripper_link_sub"/>
+  <!-- end effector link -->
+  <gazebo reference="end_effector_link">
+    <material>Gazebo/Red</material>
   </gazebo>
   <!-- ros_control plugin -->
   <gazebo>
     <plugin name="gazebo_ros_control" filename="libgazebo_ros_control.so">
-      <robotNamespace>/open_manipulator</robotNamespace>
+      <robotNamespace>open_manipulator</robotNamespace>
       <controlPeriod>0.001</controlPeriod>
       <robotSimType>gazebo_ros_control/DefaultRobotHWSim</robotSimType>

File: open_manipulator_description/urdf/open_manipulator.urdf.xacro (robot description, xacro)
@@ -6,4 +6,17 @@
   <!-- Import Rviz colors -->
   <xacro:include filename="$(find open_manipulator_description)/urdf/materials.xacro" />
+  <!-- Transmission macro -->
+  <xacro:macro name="SimpleTransmission" params="joint n">
+    <transmission name="tran${n}">
+      <type>transmission_interface/SimpleTransmission</type>
+      <joint name="${joint}">
+        <hardwareInterface>hardware_interface/PositionJointInterface</hardwareInterface>
+      </joint>
+      <actuator name="motor${n}">
+        <hardwareInterface>hardware_interface/PositionJointInterface</hardwareInterface>
+        <mechanicalReduction>1</mechanicalReduction>
+      </actuator>
+    </transmission>
+  </xacro:macro>
   <!-- World -->
   <link name="world">
@@ -30,5 +43,5 @@
       </geometry>
     </collision>
-    <inertial>
+<!--    <inertial>
       <origin xyz="0 0 0" />
       <mass value="0.082" />
@@ -36,6 +49,6 @@
                iyy="0.1" iyz="0.0"
                izz="0.1" />
-    </inertial>
-    <!-- <inertial>
+    </inertial>-->
+     <inertial>
       <origin xyz="3.0876154e-04 0.0000000e+00 -1.2176461e-04" />
       <mass value="7.9119962e-02" />
@@ -43,5 +56,5 @@
                iyy="2.1898364e-05" iyz="0.0"
                izz="1.9267361e-05" />
-    </inertial> -->
+    </inertial>
   </link>
   <!-- Joint 1 -->
@@ -51,21 +64,12 @@
     <origin xyz="0.012 0.0 0.017" rpy="0 0 0"/>
     <axis xyz="0 0 1"/>
-    <limit velocity="6.5" effort="1000" lower="${-pi*0.9}" upper="${pi*0.9}" />
+    <limit velocity="4.8" effort="1" lower="${-pi*0.9}" upper="${pi*0.9}" />
   </joint>
   <!-- Transmission 1 -->
-  <transmission name="tran1">
-    <type>transmission_interface/SimpleTransmission</type>
-    <joint name="joint1">
-      <hardwareInterface>hardware_interface/EffortJointInterface</hardwareInterface>
-    </joint>
-    <actuator name="motor1">
-      <hardwareInterface>hardware_interface/EffortJointInterface</hardwareInterface>
-      <mechanicalReduction>1</mechanicalReduction>
-    </actuator>
-  </transmission>
+  <xacro:SimpleTransmission n="1" joint="joint1" />
   <!--  Link 2 -->
   <link name="link2">
     <visual>
-      <origin xyz="0 0 0.018" rpy="0 0 0"/>
+      <origin xyz="0 0 0.019" rpy="0 0 0"/>
       <geometry>
         <mesh filename="package://open_manipulator_description/meshes/chain_link2.stl" scale="0.001 0.001 0.001"/>
@@ -74,10 +78,10 @@
     </visual>
     <collision>
-      <origin xyz="0 0 0.018" rpy="0 0 0"/>
+      <origin xyz="0 0 0.019" rpy="0 0 0"/>
       <geometry>
         <mesh filename="package://open_manipulator_description/meshes/chain_link2.stl" scale="0.001 0.001 0.001"/>
       </geometry>
     </collision>
-    <inertial>
+<!--    <inertial>
       <origin xyz="0 0 0" />
       <mass value="0.098" />
@@ -85,6 +89,6 @@
                iyy="0.1" iyz="0.0"
                izz="0.1" />
-    </inertial>
-    <!-- <inertial>
+    </inertial>-->
+     <inertial>
       <origin xyz="-3.0184870e-04 5.4043684e-04 ${0.018 + 2.9433464e-02}" />
       <mass value="9.8406837e-02" />
@@ -92,5 +96,5 @@
                iyy="3.2689329e-05" iyz="2.8511935e-08"
                izz="1.8850320e-05" />
-    </inertial> -->
+    </inertial>
   </link>
   <!--  Joint 2 -->
@@ -98,19 +102,10 @@
     <parent link="link2"/>
     <child link="link3"/>
-    <origin xyz="0.0 0.0 0.058" rpy="0 0 0"/>
+    <origin xyz="0.0 0.0 0.0595" rpy="0 0 0"/>
     <axis xyz="0 1 0"/>
-    <limit velocity="6.5" effort="1000" lower="${-pi*0.5}" upper="${pi*0.5}" />
+    <limit velocity="4.8" effort="1" lower="${-pi*0.57}" upper="${pi*0.5}" />
   </joint>
   <!-- Transmission 2 -->
-  <transmission name="tran2">
-    <type>transmission_interface/SimpleTransmission</type>
-    <joint name="joint2">
-      <hardwareInterface>hardware_interface/EffortJointInterface</hardwareInterface>
-    </joint>
-    <actuator name="motor2">
-      <hardwareInterface>hardware_interface/EffortJointInterface</hardwareInterface>
-      <mechanicalReduction>1</mechanicalReduction>
-    </actuator>
-  </transmission>
+  <xacro:SimpleTransmission n="2" joint="joint2" />
   <!--  Link 3 -->
   <link name="link3">
@@ -128,5 +123,5 @@
       </geometry>
     </collision>
-    <inertial>
+<!--    <inertial>
       <origin xyz="0 0 0" />
       <mass value="0.136" />
@@ -134,6 +129,6 @@
                iyy="0.1" iyz="0.0"
                izz="0.1" />
-    </inertial>
-    <!-- <inertial>
+    </inertial>-->
+     <inertial>
       <origin xyz="1.0308393e-02 3.7743363e-04 1.0170197e-01" />
       <mass value="1.3850917e-01" />
@@ -141,5 +136,5 @@
                iyy="3.4290447e-04" iyz="-1.5717516e-06"
                izz="6.0346498e-05" />
-    </inertial> -->
+    </inertial>
   </link>
   <!--  Joint 3 -->
@@ -149,17 +144,8 @@
     <origin xyz="0.024 0 0.128" rpy="0 0 0"/>
     <axis xyz="0 1 0"/>
-    <limit velocity="6.5" effort="1000" lower="${-pi*0.3}" upper="${pi*0.44}" />
+    <limit velocity="4.8" effort="1" lower="${-pi*0.3}" upper="${pi*0.44}" />
   </joint>
   <!-- Transmission 3 -->
-  <transmission name="tran3">
-    <type>transmission_interface/SimpleTransmission</type>
-    <joint name="joint3">
-      <hardwareInterface>hardware_interface/EffortJointInterface</hardwareInterface>
-    </joint>
-    <actuator name="motor3">
-      <hardwareInterface>hardware_interface/EffortJointInterface</hardwareInterface>
-      <mechanicalReduction>1</mechanicalReduction>
-    </actuator>
-  </transmission>
+  <xacro:SimpleTransmission n="3" joint="joint3" />
   <!--  Link 4 -->
   <link name="link4">
@@ -177,5 +163,5 @@
       </geometry>
     </collision>
-    <inertial>
+<!--    <inertial>
       <origin xyz="0 0 0" />
       <mass value="0.131" />
@@ -183,6 +169,6 @@
                iyy="0.1" iyz="0.0"
                izz="0.1" />
-    </inertial>
-    <!-- <inertial>
+    </inertial>-->
+     <inertial>
       <origin xyz="9.0909590e-02 3.8929816e-04 2.2413279e-04" />
       <mass value="1.3274562e-01" />
@@ -190,5 +176,5 @@
                iyy="2.4230292e-04" iyz="1.1559550e-08"
                izz="2.5155057e-04" />
-    </inertial> -->
+    </inertial>
   </link>
   <!--  Joint 4 -->
@@ -198,17 +184,8 @@
     <origin xyz="0.124 0.0 0.0" rpy="0 0 0"/>
     <axis xyz="0 1 0"/>
-    <limit velocity="6.5" effort="1000" lower="${-pi*0.4}" upper="${pi*0.5}" />
+    <limit velocity="4.8" effort="1" lower="${-pi*0.57}" upper="${pi*0.65}" />
   </joint>
   <!-- Transmission 4 -->
-  <transmission name="tran4">
-    <type>transmission_interface/SimpleTransmission</type>
-    <joint name="joint4">
-      <hardwareInterface>hardware_interface/EffortJointInterface</hardwareInterface>
-    </joint>
-    <actuator name="motor4">
-      <hardwareInterface>hardware_interface/EffortJointInterface</hardwareInterface>
-      <mechanicalReduction>1</mechanicalReduction>
-    </actuator>
-  </transmission>
+  <xacro:SimpleTransmission n="4" joint="joint4" />
   <!--  Link 5 -->
   <link name="link5">
@@ -226,5 +203,5 @@
       </geometry>
     </collision>
-    <inertial>
+<!--    <inertial>
       <origin xyz="0 0 0" />
       <mass value="0.141" />
@@ -232,6 +209,6 @@
                iyy="0.1" iyz="0.0"
                izz="0.1" />
-    </inertial>
-    <!-- <inertial>
+    </inertial>-->
+     <inertial>
       <origin xyz="4.4206755e-02 3.6839985e-07 8.9142216e-03" />
       <mass value="1.4327573e-01" />
@@ -239,10 +216,10 @@
                iyy="7.5980465e-05" iyz="0.0"
                izz="9.3127351e-05" />
-    </inertial> -->
-  </link>
-  <!--  Grip link -->
-  <link name="grip_link">
-    <visual>
-      <origin xyz="0.028 0.0246 0" rpy="0 0 0"/>
+    </inertial>
+  </link>
+  <!--  Gripper link -->
+  <link name="gripper_link">
+    <visual>
+      <origin xyz="0.0 0.0 0" rpy="0 0 0"/>
       <geometry>
         <mesh filename="package://open_manipulator_description/meshes/chain_link_grip_l.stl" scale="0.001 0.001 0.001"/>
@@ -251,5 +228,5 @@
     </visual>
     <collision>
-      <origin xyz="0.028 0.0246 0" rpy="0 0 0"/>
+      <origin xyz="0.0 0.0 0" rpy="0 0 0"/>
       <geometry>
         <mesh filename="package://open_manipulator_description/meshes/chain_link_grip_l.stl" scale="0.001 0.001 0.001"/>
@@ -259,9 +236,9 @@
       <origin xyz="0 0 0" />
       <mass value="0.017" />
-      <inertia ixx="0.1" ixy="0.0" ixz="0.0"
-               iyy="0.1" iyz="0.0"
-               izz="0.1" />
-    </inertial>
-    <!-- <inertial>
+      <inertia ixx="1.0e-03" ixy="0.0" ixz="0.0"
+               iyy="1.0e-03" iyz="0.0"
+               izz="1.0e-03" />
+    </inertial>
+<!--     <inertial>
       <origin xyz="${0.028 + 8.3720668e-03} ${0.0246 + 9.9696160e-03} -4.2836895e-07" />
       <mass value="3.2218127e-02" />
@@ -269,29 +246,20 @@
                iyy="2.2552871e-05" iyz="-3.1463634e-10"
                izz="1.7605306e-05" />
-    </inertial> -->
-  </link>
-  <!--  Grip joint -->
-  <joint name="grip_joint" type="prismatic">
+    </inertial>-->
+  </link>
+  <!--  Gripper joint -->
+  <joint name="gripper" type="prismatic">
     <parent link="link5"/>
-    <child link="grip_link"/>
-    <origin xyz="0.0536 0.0 0.0" rpy="0 0 0"/>
-    <axis xyz="0 -1 0"/>
-    <limit velocity="3.5" effort="100" lower="-0.015" upper="0.0105" />
+    <child link="gripper_link"/>
+    <origin xyz="0.0817 0.021 0.0" rpy="0 0 0"/>
+    <axis xyz="0 1 0"/>
+    <limit velocity="4.8" effort="1" lower="-0.010" upper="0.019" />
   </joint>
   <!-- Transmission 5 -->
-  <transmission name="tran5">
-    <type>transmission_interface/SimpleTransmission</type>
-    <joint name="grip_joint">
-      <hardwareInterface>hardware_interface/EffortJointInterface</hardwareInterface>
-    </joint>
-    <actuator name="motor7">
-      <hardwareInterface>hardware_interface/EffortJointInterface</hardwareInterface>
-      <mechanicalReduction>1</mechanicalReduction>
-    </actuator>
-  </transmission>
-  <!--  Grip link sub -->
-  <link name="grip_link_sub">
-    <visual>
-      <origin xyz="0.028 -0.0246 0" rpy="0 0 0"/>
+  <xacro:SimpleTransmission n="5" joint="gripper" />
+  <!--  Gripper link sub -->
+  <link name="gripper_link_sub">
+    <visual>
+      <origin xyz="0.0 -0.0 0" rpy="0 0 0"/>
       <geometry>
         <mesh filename="package://open_manipulator_description/meshes/chain_link_grip_r.stl" scale="0.001 0.001 0.001"/>
@@ -300,5 +268,5 @@
     </visual>
     <collision>
-      <origin xyz="0.028 -0.0246 0" rpy="0 0 0"/>
+      <origin xyz="0.0 -0.0 0" rpy="0 0 0"/>
       <geometry>
         <mesh filename="package://open_manipulator_description/meshes/chain_link_grip_r.stl" scale="0.001 0.001 0.001"/>
@@ -308,9 +276,9 @@
       <origin xyz="0 0 0" />
       <mass value="0.017" />
-      <inertia ixx="0.1" ixy="0.0" ixz="0.0"
-               iyy="0.1" iyz="0.0"
-               izz="0.1" />
-    </inertial>
-    <!-- <inertial>
+      <inertia ixx="1.0e-03" ixy="0.0" ixz="0.0"
+               iyy="1.0e-03" iyz="0.0"
+               izz="1.0e-03" />
+    </inertial>
+<!--     <inertial>
       <origin xyz="${0.028 + 8.3720668e-03} ${-0.0246 - 9.9696160e-03} -4.2836895e-07" />
       <mass value="3.2218127e-02" />
@@ -318,24 +286,37 @@
                iyy="2.2552871e-05" iyz="-3.1463634e-10"
                izz="1.7605306e-05" />
-    </inertial> -->
-  </link>
-  <!--  Grip joint sub -->
-  <joint name="grip_joint_sub" type="prismatic">
+    </inertial>-->
+  </link>
+  <!--  Gripper joint sub -->
+  <joint name="gripper_sub" type="prismatic">
     <parent link="link5"/>
-    <child link="grip_link_sub"/>
-    <origin xyz="0.0536 0 0" rpy="0 0 0"/>
-    <axis xyz="0 1 0"/>
-    <limit velocity="3.5" effort="100" lower="-0.015" upper="0.0105" />
+    <child link="gripper_link_sub"/>
+    <origin xyz="0.0817 -0.021 0" rpy="0 0 0"/>
+    <axis xyz="0 -1 0"/>
+    <limit velocity="4.8" effort="1" lower="-0.010" upper="0.019" />
+    <mimic joint="gripper" multiplier="1"/>
   </joint>
   <!-- Transmission 6 -->
-  <transmission name="tran6">
-    <type>transmission_interface/SimpleTransmission</type>
-    <joint name="grip_joint_sub">
-      <hardwareInterface>hardware_interface/EffortJointInterface</hardwareInterface>
-    </joint>
-    <actuator name="motor8">
-      <hardwareInterface>hardware_interface/EffortJointInterface</hardwareInterface>
-      <mechanicalReduction>1</mechanicalReduction>
-    </actuator>
-  </transmission>
+  <xacro:SimpleTransmission n="6" joint="gripper_sub" />
+  <!-- end effector joint -->
+  <joint name="end_effector_joint" type="fixed">
+    <origin xyz="0.126 0.0 0.0" rpy="0 0 0"/>
+    <parent link="link5"/>
+    <child link="end_effector_link"/>
+  </joint>
+  <!-- end effector link -->
+  <link name="end_effector_link">
+    <visual>
+      <origin xyz="0 0 0" rpy="0 0 0"/>
+      <geometry>
+        <box size="0.01 0.01 0.01" />
+      </geometry>
+      <material name="red"/>
+     </visual>
+    <inertial>
+      <origin xyz="0.0 0.0 0.0" rpy="0 0 0"/>
+      <mass value="0.001"/>
+      <inertia ixx="1.0e-06" ixy="0.0" ixz="0.0" iyy="1.0e-06" iyz="0.0" izz="1.0e-06" />
+    </inertial>
+  </link>
 </robot>
